File: hardware/boards/glasgow/glasgow.sch (KiCad schematic (older format))
At the start: 95 parts, among them J1 USB_C_USB2.0, SW1 RST, U1 CY7C68013A-56LTX, U15 TPD3S014, U2 CAT24M01X, U3 BL24C256A-SFRC, U30 ICE40HX8K-BG121, U36 TLV73312PQDRVR, U7 APX811-40UG-7, U8 TLV75533PDRVR, Y1 24M

Commit message: revC3: change the I2C address of DAC A to remove the address clash with the SMBus Alert Response Request (ARA)
- The SMBus Alert Response Request (ARA) is used by the INA233
- Add notes about this to the schematics
- Also store the correct footprint of the reset IC U7 in the schematics
  (was previously just in the layout and the assignment in the schematics wrong)
Parts:
- U7: footprint Package_TO_SOT_SMD:SOT-143 -> Glasgow:SOT-143
Other:
- note added: "Addr A DAC: 0001110\nAddr B DAC: 0001101\nAddr A Pull: 0100000\nAddr B Pull: 0100001\nAddr A ADC: 1000000\nAddr B ADC: 1000001\nSMBus ARA: 0001100\n"
- note removed: "Addr A DAC: 0001100\nAddr B DAC: 0001101\nAddr A Pull: 0100000\nAddr B Pull: 0100001\nAddr A ADC: 1000000\nAddr B ADC: 1000001"
Changed lines of the file:
@@
 Connection ~ 7000 950
 Text Notes 9750 2700 0    50   ~ 0
-Addr A DAC: 0001100\nAddr B DAC: 0001101\nAddr A Pull: 0100000\nAddr B Pull: 0100001\nAddr A ADC: 1000000\nAddr B ADC: 1000001
+Addr A DAC: 0001110\nAddr B DAC: 0001101\nAddr A Pull: 0100000\nAddr B Pull: 0100001\nAddr A ADC: 1000000\nAddr B ADC: 1000001\nSMBus ARA: 0001100\n
 Wire Wire Line
 	6000 5500 6400 5500
@@
 F 0 "U7" H 9146 3647 50  0000 L CNN
 F 1 "APX811-40UG-7" H 8750 3850 50  0000 L CNN
-F 2 "Package_TO_SOT_SMD:SOT-143" H 8800 3300 50  0001 L CNN
+F 2 "Glasgow:SOT-143" H 8800 3300 50  0001 L CNN
 F 3 "https://www.diodes.com/assets/Datasheets/APX811_812.pdf" H 8350 2900 50  0001 C CNN
 F 4 "ic-cat811jtbi" H 8700 3600 50  0001 C CNN "1b2-bom-key"
